Commit message: feat: Se añadieron obstáculos

File: install/share/bender_description/urdf/bender.xacro (robot description, xacro)
@@ -4,5 +4,15 @@
   <xacro:include filename="$(find bender_description)/urdf/rgbd_camera.xacro"/>
   <xacro:include filename="$(find bender_description)/urdf/ros2_control.xacro" />
+  <xacro:include filename="$(find bender_description)/urdf/obstacles.xacro" />
   <xacro:property name="epsilon" value="1e-4"/>
+  <!-- Parámetros para obstáculos configurables -->
+  <xacro:arg name="enable_obstacles" default="true"/>
+  <xacro:arg name="cylinder1_x" default="1.0"/>
+  <xacro:arg name="cylinder1_y" default="0.0"/>
+  <xacro:arg name="cylinder1_radius" default="0.3"/>
+  <xacro:property name="enable_obstacles" value="$(arg enable_obstacles)"/>
+  <xacro:property name="cylinder1_x" value="$(arg cylinder1_x)"/>
+  <xacro:property name="cylinder1_y" value="$(arg cylinder1_y)"/>
+  <xacro:property name="cylinder1_radius" value="$(arg cylinder1_radius)"/>
   <xacro:rgbd_camera
       prefix=""
@@ -712,3 +722,21 @@
     <limit effort="50" lower="${-1.570796 - epsilon}" upper="${1.570796 + epsilon}" velocity="50"/>
   </joint>
+  <!-- Obstáculos del entorno -->
+  <xacro:if value="${enable_obstacles}">
+    <!-- Cilindro rojo configurable -->
+    <xacro:obstacle_cylinder name="obstacle_cylinder_1"
+                           x="${cylinder1_x}" y="${cylinder1_y}" z="0.75"
+                           radius="${cylinder1_radius}" height="1.5"
+                           color="red"/>
+    <!-- Cilindro azul a la derecha -->
+    <xacro:obstacle_cylinder name="obstacle_cylinder_2"
+                           x="0.8" y="-0.8" z="0.5"
+                           radius="0.2" height="1.0"
+                           color="blue"/>
+    <!-- Caja verde más grande como mesa -->
+    <xacro:obstacle_box name="obstacle_box_1"
+                       x="1.5" y="1.0" z="0.4"
+                       width="1.5" depth="0.8" height="0.8"
+                       color="green"/>
+  </xacro:if>
 </robot>

File: install/share/bender_description/urdf/materials.xacro (robot description, xacro)
@@ -22,4 +22,7 @@
     <color rgba="1 0 0 0.5"/>
   </material>
+  <material name="green">
+    <color rgba="0 1 0 0.5"/>
+  </material>
   <material name="light_blue">
     <color rgba="0.6 0.8 1 1"/>
