Commit message: add: Mezclado todo con lo que hizo Mati

File: src/bender_description/urdf/bender.xacro (robot description, xacro)
@@ -8,4 +8,5 @@
       prefix=""
       camera_name="camera"
+      parent='l2h_1'
       xyz_offset="0.0435 0.03 0.160"
       rpy_offset="0 0 0"/>
@@ -671,23 +672,27 @@
     <child link="laser_1"/>
   </joint>
-  <joint name="wfr_to_base_link" type="fixed">
-    <origin xyz="0.135487 -0.164865 0.09982" rpy="0 0 0"/>
+  <joint name="wfr_to_base_link" type="continuous">
+    <origin rpy="0 0 0" xyz="0.135487 -0.164865 0.09982"/>
     <parent link="base_link"/>
     <child link="wfr_1"/>
-  </joint>
-  <joint name="wrr_to_base_link" type="fixed">
-    <origin xyz="-0.114513 -0.164865 0.09982" rpy="0 0 0"/>
+    <axis xyz="0 1 0"/>
+  </joint>
+  <joint name="wrr_to_base_link" type="continuous">
+    <origin rpy="0 0 0" xyz="-0.114513 -0.164865 0.09982"/>
     <parent link="base_link"/>
     <child link="wrr_1"/>
-  </joint>
-  <joint name="wfl_to_base_link" type="fixed">
-    <origin xyz="0.135487 0.150135 0.09982" rpy="0 0 0"/>
+    <axis xyz="0 1 0"/>
+  </joint>
+  <joint name="wfl_to_base_link" type="continuous">
+    <origin rpy="0 0 0" xyz="0.135487 0.150135 0.09982"/>
     <parent link="base_link"/>
     <child link="wfl_1"/>
-  </joint>
-  <joint name="wrl_to_base_link" type="fixed">
-    <origin xyz="-0.114513 0.150135 0.09982" rpy="0 0 0"/>
+    <axis xyz="0 1 0"/>
+  </joint>
+  <joint name="wrl_to_base_link" type="continuous">
+    <origin rpy="0 0 0" xyz="-0.114513 0.150135 0.09982"/>
     <parent link="base_link"/>
     <child link="wrl_1"/>
+    <axis xyz="0 1 0"/>
   </joint>
   <joint name="l1r_to_base_link" type="revolute">

File: src/bender_description/urdf/rgbd_camera.xacro (robot description, xacro)
@@ -130,5 +130,5 @@
         <update_rate>30</update_rate>
         <topic>${camera_name}</topic>
-        <gz_frame_id>${camera_name}</gz_frame_id>
+        <gz_frame_id>${camera_name}_link</gz_frame_id>
         <camera>
           <camera_info_topic>camera_info</camera_info_topic>

File: src/bender_description/urdf/ros2_control.xacro (robot description, xacro)
@@ -116,4 +116,25 @@
       <state_interface name="effort"/>
     </joint>
+    <!-- RUEDAS BASE -->
+    <joint name="wrl_to_base_link">
+      <command_interface name="velocity"/>
+      <state_interface name="velocity"/>
+      <state_interface name="position"/>
+    </joint>
+    <joint name="wrr_to_base_link">
+      <command_interface name="velocity"/>
+      <state_interface name="velocity"/>
+      <state_interface name="position"/>
+    </joint>
+    <joint name="wfl_to_base_link">
+      <command_interface name="velocity"/>
+      <state_interface name="velocity"/>
+      <state_interface name="position"/>
+    </joint>
+    <joint name="wfr_to_base_link">
+      <command_interface name="velocity"/>
+      <state_interface name="velocity"/>
+      <state_interface name="position"/>
+    </joint>
   </ros2_control>
   <gazebo>
